File: hardware/esp32-arduino/kicad_source/esp32-arduino.kicad_pcb (KiCad board)
At the start: 2 copper layers, 78 x 53 mm, 50 parts, among them CN1 ARDUINO, CON1 Micro_SDCard, P1 USB_OTG, Q1 Q_NMOS_GSD, Q2 Q_NMOS_GSD, SW1 TAST_VER, SW2 TAST_VER, U1 TPS383X, U2 MCP73831, U3 TPS736XX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

Commit message: updated netlist and layout
Parts:
- Q1, Q2: value Q_NMOS_GSD -> 2N7002
- R11: value 1k -> 0r
- R16, R17: value 1k -> 100R
- R18, R19, R5, R8: value 1k -> 10k
- R20, R21: value 1k -> 330k
- R7: value 1k -> 2k5
Changed lines of the file:
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@@
       (effects (font (size 1 1) (thickness 0.15)))
     )
-    (fp_text value 1k (at 0 1.9 270) (layer F.Fab)
+    (fp_text value 10k (at 0 1.9 270) (layer F.Fab)
       (effects (font (size 1 1) (thickness 0.15)))
     )
@@
       (effects (font (size 1 1) (thickness 0.15)))
     )
-    (fp_text value 1k (at 0 1.9 270) (layer F.Fab)
+    (fp_text value 2k5 (at 0 1.9 270) (layer F.Fab)
       (effects (font (size 1 1) (thickness 0.15)))
     )
@@
       (effects (font (size 1 1) (thickness 0.15)))
     )
-    (fp_text value 1k (at 0 1.9 180) (layer F.Fab)
+    (fp_text value 10k (at 0 1.9 180) (layer F.Fab)
       (effects (font (size 1 1) (thickness 0.15)))
     )
@@
       (effects (font (size 1 1) (thickness 0.15)))
     )
-    (fp_text value 1k (at 0 1.9) (layer F.Fab)
+    (fp_text value 0r (at 0 1.9) (layer F.Fab)
       (effects (font (size 1 1) (thickness 0.15)))
     )
@@
       (effects (font (size 1 1) (thickness 0.15)))
     )
-    (fp_text value Q_NMOS_GSD (at 0 2.3 180) (layer F.Fab)
+    (fp_text value 2N7002 (at 0 2.3 180) (layer F.Fab)
       (effects (font (size 1 1) (thickness 0.15)))
     )
@@
       (effects (font (size 1 1) (thickness 0.15)))
     )
-    (fp_text value Q_NMOS_GSD (at 0 2.3 180) (layer F.Fab)
+    (fp_text value 2N7002 (at 0 2.3 180) (layer F.Fab)
       (effects (font (size 1 1) (thickness 0.15)))
     )
@@
       (effects (font (size 1 1) (thickness 0.15)))
     )
-    (fp_text value 1k (at 0 1.9) (layer F.Fab)
+    (fp_text value 100R (at 0 1.9) (layer F.Fab)
       (effects (font (size 1 1) (thickness 0.15)))
     )
@@
       (effects (font (size 1 1) (thickness 0.15)))
     )
-    (fp_text value 1k (at 0 1.9) (layer F.Fab)
+    (fp_text value 100R (at 0 1.9) (layer F.Fab)
       (effects (font (size 1 1) (thickness 0.15)))
     )
@@
       (effects (font (size 1 1) (thickness 0.15)))
     )
-    (fp_text value 1k (at 0 1.9 270) (layer F.Fab)
+    (fp_text value 10k (at 0 1.9 270) (layer F.Fab)
       (effects (font (size 1 1) (thickness 0.15)))
     )
@@
       (effects (font (size 1 1) (thickness 0.15)))
     )
-    (fp_text value 1k (at 0 1.9 270) (layer F.Fab)
+    (fp_text value 10k (at 0 1.9 270) (layer F.Fab)
       (effects (font (size 1 1) (thickness 0.15)))
     )
@@
       (effects (font (size 1 1) (thickness 0.15)))
     )
-    (fp_text value 1k (at 0 1.9 180) (layer F.Fab)
+    (fp_text value 330k (at 0 1.9 180) (layer F.Fab)
       (effects (font (size 1 1) (thickness 0.15)))
     )
@@
       (effects (font (size 1 1) (thickness 0.15)))
     )
-    (fp_text value 1k (at 0 1.9 180) (layer F.Fab)
-      (effects (font (size 1 1) (thickness 0.15)))
-    )
+    (fp_text value 330k (at 0 1.9 180) (layer F.Fab)
+      (effects (font (size 1 1) (thickness 0.15)))
+    )
