File: kicad_source/sensornator.sch (KiCad schematic (older format))
At the start: 23 parts, among them CN1 ARDUINO, CON1 Micro_SDCard, SW1 TAST_VER, SW2 TAST_VER, U5 ESP32_WROOM_32, U6 ATECC608A

Commit message: updated to latest KiCAD version
Parts:
- CN1: symbol MODULE_compute:ARDUINO -> sensornator-rescue:ARDUINO-MODULE_compute
Changed lines of the file:
@@
 EESchema Schematic File Version 4
-LIBS:sensornator-cache
-EELAYER 26 0
+EELAYER 30 0
 EELAYER END
 $Descr A4 11693 8268
@@
 ARDUINO_6
 $Comp
-L MODULE_compute:ARDUINO CN1
+L sensornator-rescue:ARDUINO-MODULE_compute CN1
 U 1 1 5B0B2CBD
 P 10700 3200

Commit message: changed C9 to 10u (reset), updated schematic pdf
Parts:
- C9: value 100n -> 10u
Other:
- note added: "Copyright generationmake 2021\nsee full project documentation at https://github.com/generationmake/sensornator"
- note removed: "Copyright generationmake 2019\nsee full project documentation at http://sensornator.generationmake.de"
Changed lines of the file:
@@
 Sheet 1 3
 Title "Sensornator"
-Date "2019-04-12"
+Date "2021-01-22"
 Rev "1.1"
 Comp "generationmake"
@@
 ADC_0
 Text Notes 500  650  0    47   ~ 0
-Copyright generationmake 2019\nsee full project documentation at http://sensornator.generationmake.de
+Copyright generationmake 2021\nsee full project documentation at https://github.com/generationmake/sensornator
 Wire Wire Line
 	10500 4350 10400 4350
@@
 P 4600 3800
 F 0 "C9" H 4610 3870 50  0000 L CNN
-F 1 "100n" H 4610 3720 50  0000 L CNN
+F 1 "10u" H 4610 3720 50  0000 L CNN
 F 2 "capacitors:C_0603" H 4600 3650 50  0001 C CNN
 F 3 "" H 4600 3800 50  0000 C CNN
