File: kicad_source/sensornator.kicad_pcb (KiCad board)
At the start: 2 copper layers, 83 x 53 mm, 73 parts, among them CN1 ARDUINO, CN2 SM04B-SRSS-TB, CN3 SM04B-GHS-TB, CN4 SM04B-GHS-TB, CN5 USB_C_Receptacle_USB2.0, CON1 Micro_SDCard, Q1 2N7002, Q2 2N7002, Q3 BC847, Q4 BC847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

Commit message: added mounting pins on connectors, added labels
Parts:
- added L1: Label, generationmake:generationmake_logo, F.Cu at (86.8, 105.1)
- added L2: Label, generationmake:generationmake_logo, B.Cu at (61.7, 94.0)
- added L3: Label, Symbol:OSHW-Symbol_8.9x8mm_SilkScreen, F.Cu at (96.2, 112.4)
- added L4: Label, generationmake:opencyphal_small, F.Cu at (99.8, 85.4)
Connections:
- CN2 pad MP: (no net) -> /MP_2
- CN3 pad MP: (no net) -> /MP
- CN4 pad MP: (no net) -> /MP
Routing:
- net /MP: track 0.00 -> 23.8 mm, vias 0 -> 8
- net /ARDUINO_7: track 82.9 -> 90.7 mm
- net /MP_2: track 0.00 -> 7.40 mm, vias 0 -> 4
- net /ARDUINO_5: track 74.4 -> 81.2 mm
- net VCC: track 79.3 -> 82.0 mm
- net RESET: track 123.1 -> 124.8 mm
- net /SPI_MOSI: track 58.6 -> 60.2 mm
- net +3V3: track 255.2 -> 256.8 mm
- net /ADC_4: track 94.6 -> 95.8 mm
- net Net-(BT1-Pad1): track 9.90 -> 10.8 mm
- net /ARDUINO_6: track 100.4 -> 101.2 mm
- net /ADC_5: track 98.6 -> 99.3 mm
- net /CANH: track 37.3 -> 36.7 mm
- net /CANL: track 35.0 -> 34.5 mm
- net GND: vias 31 -> 39
